File: trafficLight.kicad_sch (KiCad schematic)
At the start: 11 parts, among them J1 Conn_01x04

Commit message: Recent modicifation of layout
i	deleted:    trafficLight-backups/trafficLight-2022-02-05_192826.zip
Parts:
- D1, D2, D3: footprint LED_THT:LED_D3.0mm -> LED_THT:LED_D5.0mm
- J1: footprint Connector:FanPinHeader_1x04_P2.54mm_Vertical -> Connector_JST:JST_PH_B4B-PH-K_1x04_P2.00mm_Vertical
- R1, R2, R3: footprint Resistor_THT:R_Axial_DIN0204_L3.6mm_D1.6mm_P5.08mm_Horizontal -> Resistor_THT:R_Axial_DIN0207_L6.3mm_D2.5mm_P10.16mm_Horizontal
Changed lines of the file:
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@@
     (property "Reference" "R2" (id 0) (at 140.97 71.12 90))
     (property "Value" "R" (id 1) (at 140.97 73.66 90))
-    (property "Footprint" "Resistor_THT:R_Axial_DIN0204_L3.6mm_D1.6mm_P5.08mm_Horizontal" (id 2) (at 140.97 79.248 90)
+    (property "Footprint" "Resistor_THT:R_Axial_DIN0207_L6.3mm_D2.5mm_P10.16mm_Horizontal" (id 2) (at 140.97 79.248 90)
       (effects (font (size 1.27 1.27)) hide)
     )
@@
     (property "Reference" "D2" (id 0) (at 157.7975 69.85 0))
     (property "Value" "LED" (id 1) (at 157.7975 72.39 0))
-    (property "Footprint" "LED_THT:LED_D3.0mm" (id 2) (at 156.21 77.47 0)
+    (property "Footprint" "LED_THT:LED_D5.0mm" (id 2) (at 156.21 77.47 0)
       (effects (font (size 1.27 1.27)) hide)
     )
-    (property "Datasheet" "~" (id 3) (at 156.21 77.47 0)
-      (effects (font (size 1.27 1.27)) hide)
-    )
+    (property "Datasheet" "~" (id 3) (at 156.21 77.47 0))
     (pin "1")
     (pin "2")
@@
     (property "Reference" "J1" (id 0) (at 121.92 62.23 0))
     (property "Value" "Conn_01x04" (id 1) (at 121.92 64.77 0))
-    (property "Footprint" "Connector:FanPinHeader_1x04_P2.54mm_Vertical" (id 2) (at 121.92 71.12 0)
+    (property "Footprint" "Connector_JST:JST_PH_B4B-PH-K_1x04_P2.00mm_Vertical" (id 2) (at 121.92 71.12 0)
       (effects (font (size 1.27 1.27)) hide)
     )
@@
     (property "Reference" "R1" (id 0) (at 140.97 60.96 90))
     (property "Value" "R" (id 1) (at 140.97 63.5 90))
-    (property "Footprint" "Resistor_THT:R_Axial_DIN0204_L3.6mm_D1.6mm_P5.08mm_Horizontal" (id 2) (at 140.97 69.088 90)
+    (property "Footprint" "Resistor_THT:R_Axial_DIN0207_L6.3mm_D2.5mm_P10.16mm_Horizontal" (id 2) (at 140.97 69.088 90)
       (effects (font (size 1.27 1.27)) hide)
     )
@@
     (pin "2")
   )
-  (symbol (lib_id "Device:LED") (at 156.21 67.31 180) (unit 1)
+  (symbol (lib_name "LED_1") (lib_id "Device:LED") (at 156.21 67.31 180) (unit 1)
     (in_bom yes) (on_board yes)
     (property "Reference" "D1" (id 0) (at 157.7975 59.69 0))
     (property "Value" "LED" (id 1) (at 157.7975 62.23 0))
-    (property "Footprint" "LED_THT:LED_D3.0mm" (id 2) (at 156.21 67.31 0)
+    (property "Footprint" "LED_THT:LED_D5.0mm" (id 2) (at 156.21 67.31 0)
       (effects (font (size 1.27 1.27)) hide)
     )
@@
     (property "Reference" "R3" (id 0) (at 140.97 81.28 90))
     (property "Value" "R" (id 1) (at 140.97 83.82 90))
-    (property "Footprint" "Resistor_THT:R_Axial_DIN0204_L3.6mm_D1.6mm_P5.08mm_Horizontal" (id 2) (at 140.97 89.408 90)
+    (property "Footprint" "Resistor_THT:R_Axial_DIN0207_L6.3mm_D2.5mm_P10.16mm_Horizontal" (id 2) (at 140.97 89.408 90)
       (effects (font (size 1.27 1.27)) hide)
     )
@@
     (property "Reference" "D3" (id 0) (at 157.7975 80.01 0))
     (property "Value" "LED" (id 1) (at 157.7975 82.55 0))
-    (property "Footprint" "LED_THT:LED_D3.0mm" (id 2) (at 156.21 87.63 0)
+    (property "Footprint" "LED_THT:LED_D5.0mm" (id 2) (at 156.21 87.63 0)
       (effects (font (size 1.27 1.27)) hide)
     )
@@
   (symbol_instances
     (path "/ba04d9a1-dad9-4fc9-9388-fc169d60a9e8"
-      (reference "D1") (unit 1) (value "LED") (footprint "LED_THT:LED_D3.0mm")
+      (reference "D1") (unit 1) (value "LED") (footprint "LED_THT:LED_D5.0mm")
     )
     (path "/6b119dbb-5ec9-4ac9-9ab0-77934a2162d6"
-      (reference "D2") (unit 1) (value "LED") (footprint "LED_THT:LED_D3.0mm")
+      (reference "D2") (unit 1) (value "LED") (footprint "LED_THT:LED_D5.0mm")
     )
     (path "/fbfe32b7-b518-40a5-88ba-e7bba955d50d"
-      (reference "D3") (unit 1) (value "LED") (footprint "LED_THT:LED_D3.0mm")
+      (reference "D3") (unit 1) (value "LED") (footprint "LED_THT:LED_D5.0mm")
     )
     (path "/547a6372-3cec-4c1b-abf4-b865b3a75f2a"
@@
     )
     (path "/aa847452-1f36-4fe5-8ab8-de7ed634d8d2"
-      (reference "J1") (unit 1) (value "Conn_01x04") (footprint "Connector:FanPinHeader_1x04_P2.54mm_Vertical")
+      (reference "J1") (unit 1) (value "Conn_01x04") (footprint "Connector_JST:JST_PH_B4B-PH-K_1x04_P2.00mm_Vertical")
     )
     (path "/ac2ad7e1-adfb-473e-8a98-ffd519050f63"
-      (reference "R1") (unit 1) (value "R") (footprint "Resistor_THT:R_Axial_DIN0204_L3.6mm_D1.6mm_P5.08mm_Horizontal")
+      (reference "R1") (unit 1) (value "R") (footprint "Resistor_THT:R_Axial_DIN0207_L6.3mm_D2.5mm_P10.16mm_Horizontal")
     )
     (path "/06ee1774-8007-4403-8997-5707829d5d38"
-      (reference "R2") (unit 1) (value "R") (footprint "Resistor_THT:R_Axial_DIN0204_L3.6mm_D1.6mm_P5.08mm_Horizontal")
+      (reference "R2") (unit 1) (value "R") (footprint "Resistor_THT:R_Axial_DIN0207_L6.3mm_D2.5mm_P10.16mm_Horizontal")
     )
     (path "/e1c4876d-9dfe-4029-97d5-34a81834594e"
-      (reference "R3") (unit 1) (value "R") (footprint "Resistor_THT:R_Axial_DIN0204_L3.6mm_D1.6mm_P5.08mm_Horizontal")
+      (reference "R3") (unit 1) (value "R") (footprint "Resistor_THT:R_Axial_DIN0207_L6.3mm_D2.5mm_P10.16mm_Horizontal")
     )
   )
