File: max31856/ADAFRUIT/KICAD/max31856/max31856.kicad_sch (KiCad schematic)
At the start: 19 parts, among them U1 MAX31856, U2 mic5225-3.3, X1 3.5mm term

Commit message: WIP
Connections:
- net +3V3: now also JP1.9; no longer JP1.8
- net DRDY: now also U1.7 (~{DRDY})
- net VDD: now also JP1.8; no longer JP1.9
- net at U1.11 (SDO): now also JP1.4; no longer JP1.5
- net at JP1.3: now also D1.1 (K); no longer D3.1 (K)
- net at D2.1 (K): now also JP1.5; no longer JP1.6
- net GNDD renamed GND
- new net: D3.1 (K), JP1.6
Other:
- moved on the sheet: C5, C7, U2, X1
